File: MSP430G2553_Controller_breadboard_kits/msp430g2553_controller_breadboard_kits.sch (EAGLE design)
At the start: 12 parts, among them J3 programmer header, U1 MSP430G2553_24IO_28PIN_TSSOP

Commit message: done the design
Parts:
- removed J3: programmer header, Connectors:4PIN_HEADER_PITCH2.54MM_TH
- added C5: 0.1uF, Capacitors:CAPACITOR_FIXED_0805
- added C6, C7, C8: (no value), Capacitors:CAPACITOR_FIXED_0805
- added R5: (no value), Resistors:RESISTOR_0805
- added U2: (no value), FTDI:FT232RL_SSOP28
- added USB1: (no value), Connectors:USB-2.0-MICRO_SMD_SMD
Connections:
- removed net P1.1: J1.3, U1.3
- removed net P1.2: J1.4, U1.4
- new net +5V: C7.1, C8.1, U2.20, USB1.VBUS
- new net DTR: C5.2, U2.2
- new net RX: J1.3, R5.2, U1.3
- new net TX: J1.4, U1.4, U2.5
- new net TXO: R5.1, U2.1
- new net USBDM: U2.16, USB1.D-
- new net USBDP: U2.15, USB1.D+
- net +3V3: now also C6.1, U2.17, U2.4; no longer J3.1
- net DGND: now also C6.2, C7.2, C8.2, D1.K, U2.18, U2.21, U2.25, U2.26, U2.7, USB1.GND, USB1.SHIELD; no longer D1.1, J3.2
- net N$2: now also D1.A; no longer D1.2
- net RST: now also C5.1; no longer J3.4
- net TEST: no longer J3.3
Other:
- moved on the sheet: BTN1, C4, D1, J1, J2, R1, R2

Commit message: update values
Parts:
- C6, C8: value (none) -> 0.1uF
- C7: value (none) -> 10uF
- R5: value (none) -> 1K
Changed lines of the file:
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@@
 <?xml version="1.0" encoding="utf-8"?>
 <!DOCTYPE eagle SYSTEM "eagle.dtd">
-<eagle version="7.7.0">
+<eagle version="8.1.0">
 <drawing>
 <settings>
@@
 <setting verticaltext="up"/>
 </settings>
-<grid distance="0.5" unitdist="mm" unit="mm" style="lines" multiple="1" display="yes" altdistance="0.01" altunitdist="inch" altunit="inch"/>
+<grid distance="0.1" unitdist="inch" unit="inch" style="lines" multiple="1" display="no" altdistance="0.01" altunitdist="inch" altunit="inch"/>
 <layers>
 <layer number="1" name="Top" color="4" fill="1" visible="no" active="no"/>
@@
 <part name="USB1" library="Connectors" deviceset="USB-2.0-MICRO" device="_SMD_SMD"/>
 <part name="U2" library="FTDI" deviceset="FT232RL" device="_SSOP28"/>
-<part name="C6" library="Capacitors" deviceset="CAPACITOR_FIXED" device="_0805"/>
-<part name="C7" library="Capacitors" deviceset="CAPACITOR_FIXED" device="_0805"/>
-<part name="C8" library="Capacitors" deviceset="CAPACITOR_FIXED" device="_0805"/>
+<part name="C6" library="Capacitors" deviceset="CAPACITOR_FIXED" device="_0805" value="0.1uF"/>
+<part name="C7" library="Capacitors" deviceset="CAPACITOR_FIXED" device="_0805" value="10uF"/>
+<part name="C8" library="Capacitors" deviceset="CAPACITOR_FIXED" device="_0805" value="0.1uF"/>
 <part name="DGND2" library="power" deviceset="DGND" device=""/>
 <part name="+3V2" library="power" deviceset="+3V3" device=""/>
 <part name="P+1" library="power" deviceset="+5V" device=""/>
-<part name="R5" library="Resistors" deviceset="RESISTOR" device="_0805"/>
+<part name="R5" library="Resistors" deviceset="RESISTOR" device="_0805" value="1K"/>
 </parts>
 <sheets>
